Commit message: update diana_description to use franka_ros2_controller

File: diana_description/robots/diana7/diana7.ros2_control.xacro (robot description, xacro)
@@ -4,8 +4,9 @@
         name="diana7_ros2_control"
         params="
-        name:=DianaSystem
-        prefix:=''
+        name
+        prefix
+        robot_ip
         use_fake_hardware:=true
-        robot_ip:=''
+        fake_sensor_commands:=true
         command_port:=1337
         state_port:=1338
@@ -13,22 +14,11 @@
         <ros2_control name="${name}" type="system">
             <hardware>
-                <plugin>
-                    diana_hardware/DianaSystem
-                </plugin>
-                <param name="use_fake_hardware">
-                    ${use_fake_hardware}
-                </param>
-                <param name="robot_ip">
-                    ${robot_ip}
-                </param>
-                <param name="command_port">
-                    ${command_port}
-                </param>
-                <param name="state_port">
-                    ${state_port}
-                </param>
-                <param name="control_frequency">
-                    ${control_frequency}
-                </param>
+                <plugin>franka_hardware/FrankaHardwareInterface</plugin>
+                <param name="version">1.0.0</param>
+                <param name="robot_ip">${robot_ip}</param>
+                <param name="robot_type">diana7</param>
+                <param name="prefix">${prefix}</param>
+                <param name="use_fake_hardware"> ${use_fake_hardware}</param>
+                <param name="fake_sensor_commands"> ${fake_sensor_commands} </param>
             </hardware>
             <!-- Joint 1 -->

File: diana_description/robots/diana7/diana7.urdf.xacro (robot description, xacro)
@@ -3,65 +3,67 @@
     xmlns:xacro="http://www.ros.org/wiki/xacro"
     name="diana7">
-  <!-- ====================================================== -->
-  <!-- Arguments                                               -->
-  <!-- ====================================================== -->
-  <xacro:arg name="prefix" default=""/>
-  <xacro:arg name="use_fake_hardware" default="true"/>
-  <xacro:arg name="fake_sensor_commands" default="false"/>
-  <xacro:arg name="use_gazebo" default="false"/>
-  <xacro:arg name="robot_ip" default=""/>
-  <xacro:arg name="command_port" default="1337"/>
-  <xacro:arg name="state_port" default="1338"/>
-  <xacro:arg name="control_frequency" default="1000"/>
-  <!-- ====================================================== -->
-  <!-- Properties                                              -->
-  <!-- ====================================================== -->
-  <xacro:property name="prefix"
-                  value="$(arg prefix)"/>
-  <xacro:property name="use_fake_hardware"
-                  value="$(arg use_fake_hardware)"/>
-  <xacro:property name="fake_sensor_commands"
-                  value="$(arg fake_sensor_commands)"/>
-  <xacro:property name="use_gazebo"
-                  value="$(arg use_gazebo)"/>
-  <xacro:property name="robot_ip"
-                  value="$(arg robot_ip)"/>
-  <xacro:property name="command_port"
-                  value="$(arg command_port)"/>
-  <xacro:property name="state_port"
-                  value="$(arg state_port)"/>
-  <xacro:property name="control_frequency"
-                  value="$(arg control_frequency)"/>
-  <!-- ====================================================== -->
-  <!-- Includes                                                -->
-  <!-- ====================================================== -->
-  <xacro:include
-      filename="$(find diana_description)/robots/diana7/diana7_arm.urdf.xacro"/>
-  <xacro:include
-      filename="$(find diana_description)/robots/diana7/diana7.ros2_control.xacro"/>
-  <xacro:include
-      filename="$(find diana_description)/robots/diana7/diana7.gazebo.xacro"/>
-  <!-- ====================================================== -->
-  <!-- Robot                                                   -->
-  <!-- ====================================================== -->
-  <xacro:diana7
-      prefix="${prefix}"/>
-  <!-- ====================================================== -->
-  <!-- ros2_control                                            -->
-  <!-- ====================================================== -->
-  <xacro:diana7_ros2_control
-      name="DianaSystem"
-      prefix="${prefix}"
-      use_fake_hardware="${use_fake_hardware}"
-      robot_ip="${robot_ip}"
-      command_port="${command_port}"
-      state_port="${state_port}"
-      control_frequency="${control_frequency}"/>
-  <!-- ====================================================== -->
-  <!-- Gazebo                                                  -->
-  <!-- ====================================================== -->
-  <xacro:if value="${use_gazebo}">
-    <xacro:diana7_gazebo
-        prefix="${prefix}"/>
-  </xacro:if>
+    <!-- ====================================================== -->
+    <!-- Arguments                                               -->
+    <!-- ====================================================== -->
+    <xacro:arg name="prefix" default="" />
+    <xacro:arg name="use_fake_hardware" default="true" />
+    <xacro:arg name="fake_sensor_commands" default="false" />
+    <xacro:arg name="use_gazebo" default="false" />
+    <xacro:arg name="robot_ip" default="192.168.10.75" />
+    <xacro:arg name="robot_type" default="diana7" />
+    <xacro:arg name="command_port" default="1337" />
+    <xacro:arg name="state_port" default="1338" />
+    <xacro:arg name="control_frequency" default="1000" />
+    <!-- ====================================================== -->
+    <!-- Properties                                              -->
+    <!-- ====================================================== -->
+    <xacro:property name="prefix"
+        value="$(arg prefix)" />
+    <xacro:property name="use_fake_hardware"
+        value="$(arg use_fake_hardware)" />
+    <xacro:property name="fake_sensor_commands"
+        value="$(arg fake_sensor_commands)" />
+    <xacro:property name="use_gazebo"
+        value="$(arg use_gazebo)" />
+    <xacro:property name="robot_ip"
+        value="$(arg robot_ip)" />
+    <xacro:property name="command_port"
+        value="$(arg command_port)" />
+    <xacro:property name="state_port"
+        value="$(arg state_port)" />
+    <xacro:property name="control_frequency"
+        value="$(arg control_frequency)" />
+    <!-- ====================================================== -->
+    <!-- Includes                                                -->
+    <!-- ====================================================== -->
+    <xacro:include
+        filename="$(find diana_description)/robots/diana7/diana7_arm.urdf.xacro" />
+    <xacro:include
+        filename="$(find diana_description)/robots/diana7/diana7.ros2_control.xacro" />
+    <xacro:include
+        filename="$(find diana_description)/robots/diana7/diana7.gazebo.xacro" />
+    <!-- ====================================================== -->
+    <!-- Robot                                                   -->
+    <!-- ====================================================== -->
+    <xacro:diana7
+        prefix="${prefix}" />
+    <!-- ====================================================== -->
+    <!-- ros2_control                                            -->
+    <!-- ====================================================== -->
+    <xacro:diana7_ros2_control
+        name="diana7_ros2_control"
+        prefix="${prefix}"
+        use_fake_hardware="${use_fake_hardware}"
+        fake_sensor_commands="${fake_sensor_commands}"
+        robot_ip="${robot_ip}"
+        command_port="${command_port}"
+        state_port="${state_port}"
+        control_frequency="${control_frequency}" />
+    <!-- ====================================================== -->
+    <!-- Gazebo                                                  -->
+    <!-- ====================================================== -->
+    <xacro:if value="${use_gazebo}">
+        <xacro:diana7_gazebo
+            prefix="${prefix}" />
+    </xacro:if>
 </robot>

Commit message: update diana7_moveit_config by using new diana_description

File: diana_description/robots/diana7/diana7.ros2_control.xacro (robot description, xacro)
@@ -7,6 +7,7 @@
         prefix
         robot_ip
-        use_fake_hardware:=true
-        fake_sensor_commands:=true
+        robot_type
+        use_fake_hardware
+        fake_sensor_commands
         command_port:=1337
         state_port:=1338
@@ -17,5 +18,5 @@
                 <param name="version">1.0.0</param>
                 <param name="robot_ip">${robot_ip}</param>
-                <param name="robot_type">diana7</param>
+                <param name="robot_type">${robot_type}</param>
                 <param name="prefix">${prefix}</param>
                 <param name="use_fake_hardware"> ${use_fake_hardware}</param>

File: diana_description/robots/diana7/diana7.urdf.xacro (robot description, xacro)
@@ -7,5 +7,5 @@
     <!-- ====================================================== -->
     <xacro:arg name="prefix" default="" />
-    <xacro:arg name="use_fake_hardware" default="true" />
+    <xacro:arg name="use_fake_hardware" default="false" />
     <xacro:arg name="fake_sensor_commands" default="false" />
     <xacro:arg name="use_gazebo" default="false" />
@@ -28,4 +28,6 @@
     <xacro:property name="robot_ip"
         value="$(arg robot_ip)" />
+    <xacro:property name="robot_type"
+        value="$(arg robot_type)" />
     <xacro:property name="command_port"
         value="$(arg command_port)" />
@@ -57,4 +59,5 @@
         fake_sensor_commands="${fake_sensor_commands}"
         robot_ip="${robot_ip}"
+        robot_type="${robot_type}"
         command_port="${command_port}"
         state_port="${state_port}"

Commit message: update diana7 description and config to keep align with Franka naming convention

File: diana_description/robots/diana7/diana7.ros2_control.xacro (robot description, xacro)
@@ -34,5 +34,5 @@
             </xacro:if>
             <!-- Joint 1 -->
-            <joint name="${prefix}joint1">
+            <joint name="${prefix}diana7_joint1">
                 <command_interface name="position" />
                 <command_interface name="velocity" />
@@ -43,5 +43,5 @@
             </joint>
             <!-- Joint 2 -->
-            <joint name="${prefix}joint2">
+            <joint name="${prefix}diana7_joint2">
                 <command_interface name="position" />
                 <command_interface name="velocity" />
@@ -52,5 +52,5 @@
             </joint>
             <!-- Joint 3 -->
-            <joint name="${prefix}joint3">
+            <joint name="${prefix}diana7_joint3">
                 <command_interface name="position" />
                 <command_interface name="velocity" />
@@ -61,5 +61,5 @@
             </joint>
             <!-- Joint 4 -->
-            <joint name="${prefix}joint4">
+            <joint name="${prefix}diana7_joint4">
                 <command_interface name="position" />
                 <command_interface name="velocity" />
@@ -70,5 +70,5 @@
             </joint>
             <!-- Joint 5 -->
-            <joint name="${prefix}joint5">
+            <joint name="${prefix}diana7_joint5">
                 <command_interface name="position" />
                 <command_interface name="velocity" />
@@ -79,5 +79,5 @@
             </joint>
             <!-- Joint 6 -->
-            <joint name="${prefix}joint6">
+            <joint name="${prefix}diana7_joint6">
                 <command_interface name="position" />
                 <command_interface name="velocity" />
@@ -88,5 +88,5 @@
             </joint>
             <!-- Joint 7 -->
-            <joint name="${prefix}joint7">
+            <joint name="${prefix}diana7_joint7">
                 <command_interface name="position" />
                 <command_interface name="velocity" />
@@ -192,5 +192,5 @@
                 <param name="index">1</param>
             </gpio>
-            <sensor name="tcp">
+            <sensor name="diana7_tcp">
                 <state_interface name="force.x" />
                 <state_interface name="force.y" />

File: diana_description/robots/diana7/diana7_arm.urdf.xacro (robot description, xacro)
@@ -92,5 +92,5 @@
         <xacro:property name="parent_link" value="${prefix}link${num-1}" />
       </xacro:unless>
-      <joint name="${prefix}joint${num}" type="revolute">
+      <joint name="${prefix}diana7_joint${num}" type="revolute">
         <xacro:dh_to_origin a="${a}" alpha="${alpha}" d="${d}" theta="${theta}" />
         <parent link="${parent_link}" />
